File: Design Files/_saved_oneMicro ATmega328.sch (KiCad schematic (older format))
At the start: 29 parts, among them CON1 USB-MINI-B, IC1 ATMEGA328P-A, IC2 MIC5205, P14 CONN_01X01, P2 CONN_01X12, P3 CONN_01X02, P5 CONN_01X12, SW1 RESET, U1 CP2102, X1 16MHz

Commit message: Design Completed
Parts:
- gave numbers to parts that had none: 1
Changed lines of the file:
@@
 $EndDescr
 $Comp
-L GND #PWR01
+L GND #PWR4
 U 1 1 57E3BD58
 P 850 2350
-F 0 "#PWR01" H 850 2100 50  0001 C CNN
+F 0 "#PWR4" H 850 2100 50  0001 C CNN
 F 1 "GND" H 850 2200 50  0000 C CNN
 F 2 "" H 850 2350 50  0000 C CNN
@@
 $EndComp
 $Comp
-L GND #PWR02
+L GND #PWR2
 U 1 1 57E3BD5C
 P 650 1400
-F 0 "#PWR02" H 650 1150 50  0001 C CNN
+F 0 "#PWR2" H 650 1150 50  0001 C CNN
 F 1 "GND" H 650 1250 50  0000 C CNN
 F 2 "" H 650 1400 50  0000 C CNN
@@
 $EndComp
 $Comp
-L GND #PWR03
+L GND #PWR13
 U 1 1 57E3BD60
 P 4500 4350
-F 0 "#PWR03" H 4500 4100 50  0001 C CNN
+F 0 "#PWR13" H 4500 4100 50  0001 C CNN
 F 1 "GND" H 4500 4200 50  0000 C CNN
 F 2 "" H 4500 4350 50  0000 C CNN
@@
 RAW
 $Comp
-L GND #PWR04
+L GND #PWR20
 U 1 1 57E438EC
 P 10300 6250
-F 0 "#PWR04" H 10300 6000 50  0001 C CNN
+F 0 "#PWR20" H 10300 6000 50  0001 C CNN
 F 1 "GND" H 10300 6100 50  0000 C CNN
 F 2 "" H 10300 6250 50  0000 C CNN
@@
 $EndComp
 $Comp
-L GND #PWR05
+L GND #PWR11
 U 1 1 57E438EF
 P 4500 1950
-F 0 "#PWR05" H 4500 1700 50  0001 C CNN
+F 0 "#PWR11" H 4500 1700 50  0001 C CNN
 F 1 "GND" H 4500 1800 50  0000 C CNN
 F 2 "" H 4500 1950 50  0000 C CNN
@@
 $EndComp
 $Comp
-L GND #PWR06
+L GND #PWR5
 U 1 1 57E438F1
 P 850 2350
-F 0 "#PWR06" H 850 2100 50  0001 C CNN
+F 0 "#PWR5" H 850 2100 50  0001 C CNN
 F 1 "GND" H 850 2200 50  0000 C CNN
 F 2 "" H 850 2350 50  0000 C CNN
@@
 $EndComp
 $Comp
-L GND #PWR07
+L GND #PWR6
 U 1 1 57E438F3
 P 1050 3650
-F 0 "#PWR07" H 1050 3400 50  0001 C CNN
+F 0 "#PWR6" H 1050 3400 50  0001 C CNN
 F 1 "GND" H 1050 3500 50  0000 C CNN
 F 2 "" H 1050 3650 50  0000 C CNN
@@
 $EndComp
 $Comp
-L GND #PWR08
+L GND #PWR3
 U 1 1 57E438F5
 P 650 1400
-F 0 "#PWR08" H 650 1150 50  0001 C CNN
+F 0 "#PWR3" H 650 1150 50  0001 C CNN
 F 1 "GND" H 650 1250 50  0000 C CNN
 F 2 "" H 650 1400 50  0000 C CNN
@@
 $EndComp
 $Comp
-L GND #PWR09
+L GND #PWR14
 U 1 1 57E438F9
 P 4500 4350
-F 0 "#PWR09" H 4500 4100 50  0001 C CNN
+F 0 "#PWR14" H 4500 4100 50  0001 C CNN
 F 1 "GND" H 4500 4200 50  0000 C CNN
 F 2 "" H 4500 4350 50  0000 C CNN
@@
 	2700 7350 2900 7350
 $Comp
-L GND #PWR010
+L GND #PWR9
 U 1 1 57E44FB2
 P 2200 7400
-F 0 "#PWR010" H 2200 7400 30  0001 C CNN
+F 0 "#PWR9" H 2200 7400 30  0001 C CNN
 F 1 "GND" H 2200 7330 30  0001 C CNN
 F 2 "" H 2200 7400 60  0001 C CNN
@@
 Connection ~ 2450 5550
 $Comp
-L GND #PWR011
+L GND #PWR7
 U 1 1 57E44FB4
 P 2150 6100
-F 0 "#PWR011" H 2150 6100 30  0001 C CNN
+F 0 "#PWR7" H 2150 6100 30  0001 C CNN
 F 1 "GND" H 2150 6030 30  0001 C CNN
 F 2 "" H 2150 6100 60  0001 C CNN
@@
 $EndComp
 $Comp
-L GND #PWR012
+L GND #PWR18
 U 1 1 57E438E9
 P 9150 5800
-F 0 "#PWR012" H 9150 5550 50  0001 C CNN
+F 0 "#PWR18" H 9150 5550 50  0001 C CNN
 F 1 "GND" H 9150 5650 50  0000 C CNN
 F 2 "" H 9150 5800 50  0000 C CNN
@@
 Open for 3.3V Board
 $Comp
-L VCC #PWR013
+L VCC #PWR19
 U 1 1 57E64412
 P 10100 5100
-F 0 "#PWR013" H 10100 4950 50  0001 C CNN
+F 0 "#PWR19" H 10100 4950 50  0001 C CNN
 F 1 "VCC" H 10100 5250 50  0000 C CNN
 F 2 "" H 10100 5100 50  0000 C CNN
@@
 $EndComp
 $Comp
-L VCC #PWR014
+L VCC #PWR1
 U 1 1 57E65034
 P 650 900
-F 0 "#PWR014" H 650 750 50  0001 C CNN
+F 0 "#PWR1" H 650 750 50  0001 C CNN
 F 1 "VCC" H 650 1050 50  0000 C CNN
 F 2 "" H 650 900 50  0000 C CNN
@@
 $EndComp
 $Comp
-L VCC #PWR016
+L VCC #PWR12
 U 1 1 57E660DE
 P 4500 3050
-F 0 "#PWR016" H 4500 2900 50  0001 C CNN
+F 0 "#PWR12" H 4500 2900 50  0001 C CNN
 F 1 "VCC" H 4500 3200 50  0000 C CNN
 F 2 "" H 4500 3050 50  0000 C CNN
@@
 $EndComp
 $Comp
-L VCC #PWR017
+L VCC #PWR16
 U 1 1 57E667D6
 P 5150 2100
-F 0 "#PWR017" H 5150 1950 50  0001 C CNN
+F 0 "#PWR16" H 5150 1950 50  0001 C CNN
 F 1 "VCC" H 5150 2250 50  0000 C CNN
 F 2 "" H 5150 2100 50  0000 C CNN
@@
 $EndComp
 $Comp
-L VCC #PWR018
+L VCC #PWR10
 U 1 1 57E67CFF
 P 2700 5450
-F 0 "#PWR018" H 2700 5300 50  0001 C CNN
+F 0 "#PWR10" H 2700 5300 50  0001 C CNN
 F 1 "VCC" H 2700 5600 50  0000 C CNN
 F 2 "" H 2700 5450 50  0000 C CNN
@@
 Connection ~ 2700 5550
 $Comp
-L VCC #PWR019
+L VCC #PWR17
 U 1 1 57E68E44
 P 7150 1950
-F 0 "#PWR019" H 7150 1800 50  0001 C CNN
+F 0 "#PWR17" H 7150 1800 50  0001 C CNN
 F 1 "VCC" H 7150 2100 50  0000 C CNN
 F 2 "" H 7150 1950 50  0000 C CNN
@@
 SCL
 $Comp
-L GND #PWR020
+L GND #PWR8
 U 1 1 57E6CE22
 P 2150 6900
-F 0 "#PWR020" H 2150 6900 30  0001 C CNN
+F 0 "#PWR8" H 2150 6900 30  0001 C CNN
 F 1 "GND" H 2150 6830 30  0001 C CNN
 F 2 "" H 2150 6900 60  0001 C CNN
@@
 RESET
 $Comp
-L CONN_01X02 P?
+L CONN_01X02 P1
 U 1 1 57E95316
 P 7400 3250
-F 0 "P?" H 7400 3400 50  0000 C CNN
+F 0 "P1" H 7400 3400 50  0000 C CNN
 F 1 "CONN_01X02" V 7500 3250 50  0000 C CNN
 F 2 "Pin_Headers:Pin_Header_Straight_1x02" H 7400 3250 50  0001 C CNN
@@
 	7600 3300 7800 3300
 $Comp
-L GND #PWR?
+L GND #PWR15
 U 1 1 57EC03BD
 P 4850 1450
-F 0 "#PWR?" H 4850 1200 50  0001 C CNN
+F 0 "#PWR15" H 4850 1200 50  0001 C CNN
 F 1 "GND" H 4850 1300 50  0000 C CNN
 F 2 "" H 4850 1450 50  0000 C CNN
