File: Design Files/oneMicro ATmega328.sch (KiCad schematic (older format))
At the start: 29 parts, among them CON1 USB-MINI-B, IC1 ATMEGA328P-A, IC2 MIC5205, P1 CONN_01X02, P14 CONN_01X01, P2 CONN_01X12, P3 CONN_01X02, P5 CONN_01X12, SW1 RESET, U1 CP2102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

Commit message: Changes Done
Parts:
- removed F1: 0.5A, Fuse_Holders_and_Fuses:Fuse_SMD1206_HandSoldering, symbol FUSE
- D1, D3: symbol LED -> LED-RESCUE-oneMicro_ATmega328
- D4: footprint Diodes_SMD:SOD-123 -> Explore:Diode_New
- SW1: symbol SW_PUSH -> SW_PUSH-RESCUE-oneMicro_ATmega328
Connections:
- net VBUS: now also D4.1 (A), JP1.1
Changed lines of the file:
@@
 EESchema Schematic File Version 2
+LIBS:oneMicro ATmega328-rescue
 LIBS:power
 LIBS:device
@@
 $EndDescr
 $Comp
-L GND #PWR4
+L GND #PWR01
 U 1 1 57E3BD58
 P 850 2350
-F 0 "#PWR4" H 850 2100 50  0001 C CNN
+F 0 "#PWR01" H 850 2100 50  0001 C CNN
 F 1 "GND" H 850 2200 50  0000 C CNN
 F 2 "" H 850 2350 50  0000 C CNN
@@
 $EndComp
 $Comp
-L GND #PWR2
+L GND #PWR02
 U 1 1 57E3BD5C
 P 650 1400
-F 0 "#PWR2" H 650 1150 50  0001 C CNN
+F 0 "#PWR02" H 650 1150 50  0001 C CNN
 F 1 "GND" H 650 1250 50  0000 C CNN
 F 2 "" H 650 1400 50  0000 C CNN
@@
 $EndComp
 $Comp
-L GND #PWR13
+L GND #PWR03
 U 1 1 57E3BD60
 P 4500 4350
-F 0 "#PWR13" H 4500 4100 50  0001 C CNN
+F 0 "#PWR03" H 4500 4100 50  0001 C CNN
 F 1 "GND" H 4500 4200 50  0000 C CNN
 F 2 "" H 4500 4350 50  0000 C CNN
@@
 Connection ~ 9150 5750
 $Comp
-L LED D1
+L LED-RESCUE-oneMicro_ATmega328 D1
 U 1 1 57E3BD73
 P 4050 1400
@@
 RAW
 $Comp
-L GND #PWR20
+L GND #PWR04
 U 1 1 57E438EC
 P 10300 6250
-F 0 "#PWR20" H 10300 6000 50  0001 C CNN
+F 0 "#PWR04" H 10300 6000 50  0001 C CNN
 F 1 "GND" H 10300 6100 50  0000 C CNN
 F 2 "" H 10300 6250 50  0000 C CNN
@@
 $EndComp
 $Comp
-L GND #PWR11
+L GND #PWR05
 U 1 1 57E438EF
 P 4500 1950
-F 0 "#PWR11" H 4500 1700 50  0001 C CNN
+F 0 "#PWR05" H 4500 1700 50  0001 C CNN
 F 1 "GND" H 4500 1800 50  0000 C CNN
 F 2 "" H 4500 1950 50  0000 C CNN
@@
 $EndComp
 $Comp
-L GND #PWR5
+L GND #PWR06
 U 1 1 57E438F1
 P 850 2350
-F 0 "#PWR5" H 850 2100 50  0001 C CNN
+F 0 "#PWR06" H 850 2100 50  0001 C CNN
 F 1 "GND" H 850 2200 50  0000 C CNN
 F 2 "" H 850 2350 50  0000 C CNN
@@
 $EndComp
 $Comp
-L GND #PWR6
+L GND #PWR07
 U 1 1 57E438F3
 P 1050 3650
-F 0 "#PWR6" H 1050 3400 50  0001 C CNN
+F 0 "#PWR07" H 1050 3400 50  0001 C CNN
 F 1 "GND" H 1050 3500 50  0000 C CNN
 F 2 "" H 1050 3650 50  0000 C CNN
@@
 $EndComp
 $Comp
-L GND #PWR3
+L GND #PWR08
 U 1 1 57E438F5
 P 650 1400
-F 0 "#PWR3" H 650 1150 50  0001 C CNN
+F 0 "#PWR08" H 650 1150 50  0001 C CNN
 F 1 "GND" H 650 1250 50  0000 C CNN
 F 2 "" H 650 1400 50  0000 C CNN
@@
 $EndComp
 $Comp
-L SW_PUSH SW1
+L SW_PUSH-RESCUE-oneMicro_ATmega328 SW1
 U 1 1 57E438F7
 P 4500 4000
@@
 $EndComp
 $Comp
-L GND #PWR14
+L GND #PWR09
 U 1 1 57E438F9
 P 4500 4350
-F 0 "#PWR14" H 4500 4100 50  0001 C CNN
+F 0 "#PWR09" H 4500 4100 50  0001 C CNN
 F 1 "GND" H 4500 4200 50  0000 C CNN
 F 2 "" H 4500 4350 50  0000 C CNN
@@
 	2700 7350 2900 7350
 $Comp
-L GND #PWR9
+L GND #PWR010
 U 1 1 57E44FB2
 P 2200 7400
-F 0 "#PWR9" H 2200 7400 30  0001 C CNN
+F 0 "#PWR010" H 2200 7400 30  0001 C CNN
 F 1 "GND" H 2200 7330 30  0001 C CNN
 F 2 "" H 2200 7400 60  0001 C CNN
@@
 Connection ~ 2450 5550
 $Comp
-L GND #PWR7
+L GND #PWR011
 U 1 1 57E44FB4
 P 2150 6100
-F 0 "#PWR7" H 2150 6100 30  0001 C CNN
+F 0 "#PWR011" H 2150 6100 30  0001 C CNN
 F 1 "GND" H 2150 6030 30  0001 C CNN
 F 2 "" H 2150 6100 60  0001 C CNN
@@
 $EndComp
 $Comp
-L GND #PWR18
+L GND #PWR012
 U 1 1 57E438E9
 P 9150 5800
-F 0 "#PWR18" H 9150 5550 50  0001 C CNN
+F 0 "#PWR012" H 9150 5550 50  0001 C CNN
 F 1 "GND" H 9150 5650 50  0000 C CNN
 F 2 "" H 9150 5800 50  0000 C CNN
@@
 Text Label 2050 6400 0    60   ~ 0
 VBUS
-Text Label 6150 5050 0    60   ~ 0
+Text Label 6900 5050 2    60   ~ 0
 VBUS
-$Comp
-L FUSE F1
-U 1 1 57E5EB2C
-P 6650 5050
-F 0 "F1" H 6750 5100 50  0000 C CNN
-F 1 "0.5A" H 6650 4900 50  0000 C CNN
-F 2 "Fuse_Holders_and_Fuses:Fuse_SMD1206_HandSoldering" H 6650 5050 50  0001 C CNN
-F 3 "" H 6650 5050 50  0000 C CNN
-	1    6650 5050
-	1    0    0    -1
-$EndComp
-Wire Wire Line
-	6400 5050 6150 5050
 $Comp
 L Jumper_NC_Small JP1
@@
 F 0 "D4" H 7550 5150 40  0000 C CNN
 F 1 "DIODE" H 7550 4950 40  0000 C CNN
-F 2 "Diodes_SMD:SOD-123" H 7550 5050 60  0001 C CNN
+F 2 "Explore:Diode_New" H 7550 5050 60  0001 C CNN
 F 3 "" H 7550 5050 60  0000 C CNN
 	1    7550 5050
@@
 Open for 3.3V Board
 $Comp
-L VCC #PWR19
+L VCC #PWR013
 U 1 1 57E64412
 P 10100 5100
-F 0 "#PWR19" H 10100 4950 50  0001 C CNN
+F 0 "#PWR013" H 10100 4950 50  0001 C CNN
 F 1 "VCC" H 10100 5250 50  0000 C CNN
 F 2 "" H 10100 5100 50  0000 C CNN
@@
 $EndComp
 $Comp
-L VCC #PWR1
+L VCC #PWR014
 U 1 1 57E65034
 P 650 900
-F 0 "#PWR1" H 650 750 50  0001 C CNN
+F 0 "#PWR014" H 650 750 50  0001 C CNN
 F 1 "VCC" H 650 1050 50  0000 C CNN
 F 2 "" H 650 900 50  0000 C CNN
@@
 $EndComp
 $Comp
-L VCC #PWR12
+L VCC #PWR015
 U 1 1 57E660DE
 P 4500 3050
-F 0 "#PWR12" H 4500 2900 50  0001 C CNN
+F 0 "#PWR015" H 4500 2900 50  0001 C CNN
 F 1 "VCC" H 4500 3200 50  0000 C CNN
 F 2 "" H 4500 3050 50  0000 C CNN
@@
 $EndComp
 $Comp
-L VCC #PWR16
+L VCC #PWR016
 U 1 1 57E667D6
 P 5150 2100
-F 0 "#PWR16" H 5150 1950 50  0001 C CNN
+F 0 "#PWR016" H 5150 1950 50  0001 C CNN
 F 1 "VCC" H 5150 2250 50  0000 C CNN
 F 2 "" H 5150 2100 50  0000 C CNN
@@
 $EndComp
 $Comp
-L VCC #PWR10
+L VCC #PWR017
 U 1 1 57E67CFF
 P 2700 5450
-F 0 "#PWR10" H 2700 5300 50  0001 C CNN
+F 0 "#PWR017" H 2700 5300 50  0001 C CNN
 F 1 "VCC" H 2700 5600 50  0000 C CNN
 F 2 "" H 2700 5450 50  0000 C CNN
@@
 Connection ~ 2700 5550
 $Comp
-L VCC #PWR17
+L VCC #PWR018
 U 1 1 57E68E44
 P 7150 1950
-F 0 "#PWR17" H 7150 1800 50  0001 C CNN
+F 0 "#PWR018" H 7150 1800 50  0001 C CNN
 F 1 "VCC" H 7150 2100 50  0000 C CNN
 F 2 "" H 7150 1950 50  0000 C CNN
@@
 SCL
 $Comp
-L GND #PWR8
+L GND #PWR019
 U 1 1 57E6CE22
 P 2150 6900
-F 0 "#PWR8" H 2150 6900 30  0001 C CNN
+F 0 "#PWR019" H 2150 6900 30  0001 C CNN
 F 1 "GND" H 2150 6830 30  0001 C CNN
 F 2 "" H 2150 6900 60  0001 C CNN
@@
 VCC = 5V or 3.3V
 $Comp
-L LED D3
+L LED-RESCUE-oneMicro_ATmega328 D3
 U 1 1 57E438EA
 P 10300 5450
@@
 	7600 3300 7800 3300
 $Comp
-L GND #PWR15
+L GND #PWR020
 U 1 1 57EC03BD
 P 4850 1450
-F 0 "#PWR15" H 4850 1200 50  0001 C CNN
+F 0 "#PWR020" H 4850 1200 50  0001 C CNN
 F 1 "GND" H 4850 1300 50  0000 C CNN
 F 2 "" H 4850 1450 50  0000 C CNN
